Commit message: configure the world

File: universal_robot/ur_description/urdf_robotiq/common.gazebo.xacro (robot description, xacro)
@@ -5,4 +5,6 @@
       <!--robotNamespace>/</robotNamespace-->
       <!--robotSimType>gazebo_ros_control/DefaultRobotHWSim</robotSimType-->
+    <robotSimType>gazebo_ros_control/DefaultRobotHWSim</robotSimType>
+    <legacyModeNS>true</legacyModeNS>
     </plugin>
 <!--
@@ -21,3 +23,64 @@
 -->
   </gazebo>
+  <gazebo reference="camera_link">
+    <sensor type="depth" name="fixed_camera">
+      <always_on>true</always_on>
+      <visualize>true</visualize>
+      <camera>
+          <horizontal_fov>1.047</horizontal_fov>
+          <image>
+              <width>640</width>
+              <height>480</height>
+              <format>R8G8B8</format>
+          </image>
+          <depth_camera>
+          </depth_camera>
+          <clip>
+              <near>0.1</near>
+              <far>100</far>
+          </clip>
+      </camera>
+      <plugin name="camera_controller" filename="libgazebo_ros_openni_kinect.so">
+          <baseline>0.2</baseline>
+          <alwaysOn>true</alwaysOn>
+              <updateRate>10.0</updateRate>
+              <cameraName>fixed_camera</cameraName>
+              <frameName>camera_link</frameName>
+          <imageTopicName>fixed_camera/rgb/image_raw</imageTopicName>
+          <depthImageTopicName>fixed_camera/depth/image_raw</depthImageTopicName>
+          <pointCloudTopicName>fixed_camera/depth/points</pointCloudTopicName>
+          <cameraInfoTopicName>fixed_camera/rgb/camera_info</cameraInfoTopicName>
+          <depthImageCameraInfoTopicName>fixed_camera/depth/camera_info</depthImageCameraInfoTopicName>
+          <pointCloudCutoff>0.4</pointCloudCutoff>
+              <hackBaseline>0.07</hackBaseline>
+              <distortionK1>0.0</distortionK1>
+              <distortionK2>0.0</distortionK2>
+              <distortionK3>0.0</distortionK3>
+              <distortionT1>0.0</distortionT1>
+              <distortionT2>0.0</distortionT2>
+          <CxPrime>0.0</CxPrime>
+          <Cx>0.0</Cx>
+          <Cy>0.0</Cy>
+          <focalLength>0.0</focalLength>
+          </plugin>
+    </sensor>
+  </gazebo>
+  <gazebo reference="robotiq_arg2f_base_link">
+    <mu1>0.9</mu1>
+    <mu2>0.9</mu2>
+    <material>Gazebo/FlatBlack</material>
+  </gazebo>
+  <!-- Gazebo grasping plugin -->
+  <gazebo>
+    <gripper name="gazebo_gripper">
+      <grasp_check>
+        <attach_steps>2</attach_steps>    <!-- default: 20 -->
+        <detach_steps>2</detach_steps>    <!-- default: 40 -->
+        <min_contact_count>3</min_contact_count>
+      </grasp_check>
+      <gripper_link>left_outer_knuckle</gripper_link>
+      <gripper_link>right_outer_knuckle</gripper_link>
+      <palm_link>robotiq_arg2f_base_link</palm_link>
+    </gripper>
+  </gazebo>
 </robot>

File: universal_robot/ur_description/urdf_robotiq/ur.transmission.xacro (robot description, xacro)
@@ -5,5 +5,5 @@
       <type>transmission_interface/SimpleTransmission</type>
       <joint name="${prefix}shoulder_pan_joint">
-        <hardwareInterface>PositionJointInterface</hardwareInterface>
+        <hardwareInterface>hardware_interface/PositionJointInterface</hardwareInterface>
       </joint>
       <actuator name="${prefix}shoulder_pan_motor">
@@ -14,5 +14,5 @@
       <type>transmission_interface/SimpleTransmission</type>
       <joint name="${prefix}shoulder_lift_joint">
-        <hardwareInterface>PositionJointInterface</hardwareInterface>
+        <hardwareInterface>hardware_interface/PositionJointInterface</hardwareInterface>
       </joint>
       <actuator name="${prefix}shoulder_lift_motor">
@@ -23,5 +23,5 @@
       <type>transmission_interface/SimpleTransmission</type>
       <joint name="${prefix}elbow_joint">
-        <hardwareInterface>PositionJointInterface</hardwareInterface>
+        <hardwareInterface>hardware_interface/PositionJointInterface</hardwareInterface>
       </joint>
       <actuator name="${prefix}elbow_motor">
@@ -32,5 +32,5 @@
       <type>transmission_interface/SimpleTransmission</type>
       <joint name="${prefix}wrist_1_joint">
-        <hardwareInterface>PositionJointInterface</hardwareInterface>
+        <hardwareInterface>hardware_interface/PositionJointInterface</hardwareInterface>
       </joint>
       <actuator name="${prefix}wrist_1_motor">
@@ -41,5 +41,5 @@
       <type>transmission_interface/SimpleTransmission</type>
       <joint name="${prefix}wrist_2_joint">
-        <hardwareInterface>PositionJointInterface</hardwareInterface>
+        <hardwareInterface>hardware_interface/PositionJointInterface</hardwareInterface>
       </joint>
       <actuator name="${prefix}wrist_2_motor">
@@ -50,5 +50,5 @@
       <type>transmission_interface/SimpleTransmission</type>
       <joint name="${prefix}wrist_3_joint">
-        <hardwareInterface>PositionJointInterface</hardwareInterface>
+        <hardwareInterface>hardware_interface/PositionJointInterface</hardwareInterface>
       </joint>
       <actuator name="${prefix}wrist_3_motor">

File: universal_robot/ur_description/urdf_robotiq/ur5_joint_limited_gripper.urdf.xacro (robot description, xacro)
@@ -23,9 +23,4 @@
     <child link="robotiq_arg2f_base_link"/>
   </joint>
-  <gazebo reference="robotiq_arg2f_base_link">
-    <mu1>0.9</mu1>
-    <mu2>0.9</mu2>
-    <material>Gazebo/FlatBlack</material>
-  </gazebo>
   <!-- Gazebo FT sensor plugin -->
   <!--gazebo reference="wrist_3_joint">
@@ -40,16 +35,15 @@
     </plugin>
   </gazebo-->
-  <!-- Gazebo grasping plugin -->
-  <gazebo>
-    <gripper name="gazebo_gripper">
-      <grasp_check>
-        <attach_steps>2</attach_steps>    <!-- default: 20 -->
-        <detach_steps>2</detach_steps>    <!-- default: 40 -->
-        <min_contact_count>3</min_contact_count>
-      </grasp_check>
-      <gripper_link>left_outer_knuckle</gripper_link>
-      <gripper_link>right_outer_knuckle</gripper_link>
-      <palm_link>robotiq_arg2f_base_link</palm_link>
-    </gripper>
-  </gazebo>
+  <link name="camera_link">
+    <visual>
+      <geometry>
+      <mesh filename="package://ur_description/meshes/kinect/meshes/kinect.dae"/>
+      </geometry>
+    </visual>
+  </link>
+  <joint name="camera_joint" type="fixed">
+    <parent link="base_link" />
+    <child link = "camera_link" />
+    <origin xyz="0.0 0.0 2.0" rpy="0.0 ${pi/2} 0.0" />
+  </joint>
 </robot>

Commit message: Solve the point cloud2

File: universal_robot/ur_description/urdf_robotiq/common.gazebo.xacro (robot description, xacro)
@@ -46,5 +46,5 @@
               <updateRate>10.0</updateRate>
               <cameraName>fixed_camera</cameraName>
-              <frameName>camera_link</frameName>
+              <frameName>points_frame</frameName>
           <imageTopicName>/rgb/image_raw</imageTopicName>
           <depthImageTopicName>/depth/image_raw</depthImageTopicName>

File: universal_robot/ur_description/urdf_robotiq/ur5_simul_gripper.urdf.xacro (robot description, xacro)
@@ -88,3 +88,10 @@
     <origin xyz="0.0 0.0 2.0" rpy="0.0 ${pi/2} 0.0" />
   </joint>
+  <link name="points_frame">
+  </link>
+  <joint name="point_joint" type="fixed">
+    <parent link="camera_link" />
+    <child link = "points_frame" />
+    <origin xyz="0.0 0.0 0.0" rpy="${pi/2} ${pi} ${pi/2}" />
+  </joint>
 </robot>
